Commit message: Update rbvogui_std.urdf.xacro

File: rbvogui_description/robots/rbvogui_std.urdf.xacro (robot description, xacro)
@@ -76,5 +76,5 @@
     <!-- Camera -->
     <xacro:sensor_camera prefix="${prefix}" parent="${tf_prefix}arm_tool0">
-      <origin xyz="0.0 0.0 0.0" rpy="0 -1.57 1.57"/>
+      <origin xyz="0.0 0.0 0.0" rpy="3.14 -1.57 1.57"/>
     </xacro:sensor_camera>
     <xacro:lidar_gazebo_sensor parent="${prefix}base_link"/>
