Commit message: Update camera.urdf.xacro

File: rbvogui_description/urdf/camera/camera.urdf.xacro (robot description, xacro)
@@ -39,5 +39,5 @@
       <parent link="${prefix}camera_link"/>
       <child link="${prefix}camera_link_optical"/>
-      <origin rpy="${-pi/2} 0 ${-pi/2}" xyz="0.0 0.0 0.000" />
+      <origin rpy="${pi/2} ${pi/2} ${-pi/2}" xyz="0.0 0.0 0.000" />
     </joint>
     <link name="${prefix}camera_link_optical"/>
